File: funcoid1.sch (KiCad schematic (older format))
At the start: 36 parts, among them J1 7-15V DC, J2 NMI_CTRL, J3 IRQ_CTRL, J4 BREAKOUT, J5 S1_SERIAL, SW1 SW_RST, U1 74HC132, U2 HM62256ALP-10, U3 WD65C02, U4 W65C51N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

Commit message: Update to KiCad 5
Not sure if all the right files are here. Fingers crossed.
Parts:
- C1, C10, C9: symbol CP1_Small -> funcoid1-rescue:CP1_Small
- C2, C3, C4, C5, C6, C7, C8: symbol C_Small -> funcoid1-rescue:C_Small
- D1, D2: symbol D -> funcoid1-rescue:D
- D3: symbol LED -> funcoid1-rescue:LED
- J1: symbol Barrel_Jack -> funcoid1-rescue:Barrel_Jack
- J2: symbol Conn_01x02_Male -> funcoid1-rescue:Conn_01x02_Male
- J3: symbol Conn_01x04_Male -> funcoid1-rescue:Conn_01x04_Male
- J4: symbol Conn_02x20_Odd_Even -> funcoid1-rescue:Conn_02x20_Odd_Even
- J5: symbol DB9_Male -> funcoid1-rescue:DB9_Male
- R1, R2, R3, R4, R5, R6, R7, R8, R9: symbol R -> funcoid1-rescue:R
- SW1: symbol SW_Push -> funcoid1-rescue:SW_Push
- U1: symbol 74LS132 -> funcoid1-rescue:74LS132
- U2: symbol HM62256BLP-7 -> funcoid1-rescue:HM62256BLP-7
- U3: symbol WD65C02 -> funcoid1-rescue:WD65C02
- U4: symbol W65C51N -> funcoid1-rescue:W65C51N
- U5: symbol 28C256 -> funcoid1-rescue:28C256
- U6: symbol LM1117-5.0 -> funcoid1-rescue:LM1117-5.0
- X1: symbol ACO-xxxMHz -> funcoid1-rescue:ACO-xxxMHz
- Y1: symbol Crystal_Small -> funcoid1-rescue:Crystal_Small

Commit message: Add a MAX232 for proper RS-232 signalling
Use a MAX232 to drive the signal on the DB9 connector, such that it is
RS-232 compliant and will be understood by my VT510 terminal. Route the
old 5V CMOS UART to a new 6-pin header for use with an FTDI.

This change also moves the DB9 connector to the same edge as the barrel
jack, which should make designing a box a little easier.

Finally, do some general re-routing on the PCB layout.
Parts:
- added C11, C12, C13, C14, C15: 1u, Capacitor_THT:C_Disc_D5.0mm_W2.5mm_P5.00mm, symbol funcoid1-rescue:CP1_Small
- added J6: S1_CMOS, Connector_PinHeader_2.54mm:PinHeader_1x06_P2.54mm_Horizontal, symbol Connector:Conn_01x06_Male
- added J7: 5V DC, Connector_PinHeader_2.54mm:PinHeader_1x02_P2.54mm_Vertical, symbol Connector:Conn_01x02_Male
- added U7: MAX232_Small, Package_DIP:DIP-16_W7.62mm_Socket, symbol custom:MAX232_Small
- C1: footprint Capacitors_ThroughHole:CP_Radial_D5.0mm_P2.50mm -> Capacitor_THT:CP_Radial_D5.0mm_P2.50mm
- C10, C2, C3, C4, C5, C6, C7, C8, C9: footprint Capacitors_ThroughHole:C_Disc_D5.0mm_W2.5mm_P5.00mm -> Capacitor_THT:C_Disc_D5.0mm_W2.5mm_P5.00mm
- J5: value S1_SERIAL -> S1_RS232
- U4: symbol funcoid1-rescue:W65C51N -> custom:W65C51N_Fixed
Connections:
- net GND: now also C13.1, C14.2, C15.2, J6.1 (Pin_1), J7.1 (Pin_1), U7.15 (GND)
- net S1_CTS: now also J6.2 (Pin_2); no longer J5.8
- net S1_DCD: no longer J5.1
- net S1_DSR: no longer J5.6
- net S1_DTR: no longer J5.4
- net S1_RTS: now also J6.6 (Pin_6); no longer J5.7
- net S1_RX: now also J6.5 (Pin_5), U7.12 (R1OUT); no longer J5.2
- net S1_TX: now also J6.4 (Pin_4), U7.11 (T1IN); no longer J5.3
- net VCC: now also C15.1, J6.3 (Pin_3), J7.2 (Pin_2), U7.16 (VCC)
- new net: J5.2, U7.13 (R1IN)
- new net: J5.3, U7.14 (T1OUT)
- new net: C14.1, U7.2 (VS+)
- new net: C11.1, U7.1 (C1+)
- new net: C11.2, U7.3 (C1-)
- new net: C12.1, U7.4 (C2+)
- new net: C12.2, U7.5 (C2-)
- new net: C13.2, U7.6 (VS-)
- no-connect marks 8 -> 20
Other:
- note added: "At U7"
- moved on the sheet: C8, J5, U2, U4, Y1
